File: openlst/openlst-hw.kicad_sch (KiCad schematic)
At the start: 84 parts, among them J1 Battery, J2 CC Prog/Debug, J3 UART0, J4 SPI0, J5 Control Outputs, J6 ANT, U1 LP2981-3.3, U2 CC1110, U3 AP6502, U4 ASFL1-27.000MHZ, U5 APX803S00, U6 PE4250, U8 SF2446E, U9 RFFM6404

Commit message: Finalized BOM
Parts:
- added L2: Z=1k @ 100M, Inductor_SMD:L_0603_1608Metric, symbol openlst-hw:Ferrite_Bead
- C23, C24: Manuf Samsung -> Yageo; ManufPN CL05C3R9CB5NNNC -> AC0402CRNPO9BN3R9; SupplierPN 1276-1695-1-ND -> 311-3054-1-ND
- J6: SupplierPN (none) -> SMA-J-P-H-ST-EM1
- U5: value APX803S00 -> MIC803; Manuf Diodes Inc -> Microchip; ManufPN APX803S00-29SR-7 -> MIC803-29D3VM3-TR; SupplierPN APX803S00-29SR-7DICT-ND -> 576-3804-1-ND
- U8: Supplier Digikey Marketplace -> Mouser
Connections:
- net VAA: now also L2.1; no longer C11.1, C44.1, C46.1, C8.1, U9.17 (VCC_RX), U9.26 (VCC_TX)
- new net: C11.1, C44.1, C46.1, C8.1, L2.2, U9.17 (VCC_RX), U9.26 (VCC_TX)
Other:
- moved on the sheet: R26
Changed lines of the file:
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@@
   (title_block
     (title "OpenLST Reference Design")
-    (date "2021-07-11")
+    (date "2021-07-15")
     (rev "2.5")
     (comment 1 "Drawn by Ryan Kingsbury, Modified by Nathan Kerns")
@@
     (stroke (width 0) (type solid) (color 0 0 0 0))
   )
-  (wire (pts (xy 157.48 99.06) (xy 176.53 99.06))
-    (stroke (width 0) (type solid) (color 0 0 0 0))
-  )
   (wire (pts (xy 160.02 68.58) (xy 160.02 76.2))
     (stroke (width 0) (type solid) (color 0 0 0 0))
@@
     (stroke (width 0) (type solid) (color 0 0 0 0))
   )
+  (wire (pts (xy 167.64 99.06) (xy 176.53 99.06))
+    (stroke (width 0) (type solid) (color 0 0 0 0))
+  )
   (wire (pts (xy 167.64 101.6) (xy 167.64 104.14))
     (stroke (width 0) (type solid) (color 0 0 0 0))
@@
     (stroke (width 0) (type solid) (color 0 0 0 0))
   )
+  (wire (pts (xy 250.19 35.56) (xy 250.19 38.1))
+    (stroke (width 0) (type solid) (color 0 0 0 0))
+  )
   (wire (pts (xy 250.19 45.72) (xy 250.19 48.26))
     (stroke (width 0) (type solid) (color 0 0 0 0))
@@
     (pin "1")
   )
-  (symbol (lib_id "openlst-hw:+3.3V") (at 149.86 99.06 90) (unit 1)
+  (symbol (lib_id "openlst-hw:+3.3V") (at 160.02 99.06 90) (unit 1)
     (in_bom yes) (on_board yes)
-    (property "Reference" "#PWR0101" (id 0) (at 153.67 99.06 0)
+    (property "Reference" "#PWR0101" (id 0) (at 163.83 99.06 0)
       (effects (font (size 1.27 1.27)) hide)
     )
-    (property "Value" "+3.3V" (id 1) (at 146.304 99.06 0))
-    (property "Footprint" "" (id 2) (at 149.86 99.06 0)
+    (property "Value" "+3.3V" (id 1) (at 156.464 99.06 0))
+    (property "Footprint" "" (id 2) (at 160.02 99.06 0)
       (effects (font (size 1.27 1.27)) hide)
     )
-    (property "Datasheet" "" (id 3) (at 149.86 99.06 0)
+    (property "Datasheet" "" (id 3) (at 160.02 99.06 0)
       (effects (font (size 1.27 1.27)) hide)
     )
@@
     (pin "1")
   )
-  (symbol (lib_id "power:VAA") (at 250.19 45.72 0) (unit 1)
+  (symbol (lib_id "power:VAA") (at 250.19 35.56 0) (unit 1)
     (in_bom yes) (on_board yes)
-    (property "Reference" "#PWR021" (id 0) (at 250.19 49.53 0)
+    (property "Reference" "#PWR021" (id 0) (at 250.19 39.37 0)
       (effects (font (size 1.27 1.27)) hide)
     )
-    (property "Value" "VAA" (id 1) (at 250.19 41.91 0))
-    (property "Footprint" "" (id 2) (at 250.19 45.72 0)
+    (property "Value" "VAA" (id 1) (at 250.19 31.75 0))
+    (property "Footprint" "" (id 2) (at 250.19 35.56 0)
       (effects (font (size 1.27 1.27)) hide)
     )
-    (property "Datasheet" "" (id 3) (at 250.19 45.72 0)
+    (property "Datasheet" "" (id 3) (at 250.19 35.56 0)
       (effects (font (size 1.27 1.27)) hide)
     )
@@
     (pin "2")
   )
-  (symbol (lib_id "openlst-hw:R") (at 153.67 99.06 270) (unit 1)
-    (in_bom yes) (on_board yes)
-    (property "Reference" "R26" (id 0) (at 153.67 101.092 90))
-    (property "Value" "1k" (id 1) (at 153.67 99.06 90))
-    (property "Footprint" "Resistor_SMD:R_0603_1608Metric" (id 2) (at 153.67 97.282 90)
-      (effects (font (size 1.27 1.27)) hide)
-    )
-    (property "Datasheet" "" (id 3) (at 153.67 99.06 0)
-      (effects (font (size 1.27 1.27)) hide)
-    )
-    (property "Manuf" "Yageo" (id 4) (at 156.21 101.092 0)
-      (effects (font (size 1.27 1.27)) hide)
-    )
-    (property "ManufPN" "RC0603FR-071KL" (id 5) (at 156.21 101.092 0)
-      (effects (font (size 1.27 1.27)) hide)
-    )
-    (property "Supplier" "Digikey" (id 6) (at 156.21 101.092 0)
-      (effects (font (size 1.27 1.27)) hide)
-    )
-    (property "SupplierPN" "311-1.00KHRCT-ND" (id 7) (at 156.21 101.092 0)
-      (effects (font (size 1.27 1.27)) hide)
-    )
-    (pin "1")
-    (pin "2")
-  )
   (symbol (lib_id "openlst-hw:R") (at 161.29 137.16 180) (unit 1)
     (in_bom yes) (on_board yes)
@@
     (pin "2")
   )
+  (symbol (lib_id "openlst-hw:R") (at 163.83 99.06 270) (unit 1)
+    (in_bom yes) (on_board yes)
+    (property "Reference" "R26" (id 0) (at 163.83 101.092 90))
+    (property "Value" "1k" (id 1) (at 163.83 99.06 90))
+    (property "Footprint" "Resistor_SMD:R_0603_1608Metric" (id 2) (at 163.83 97.282 90)
+      (effects (font (size 1.27 1.27)) hide)
+    )
+    (property "Datasheet" "" (id 3) (at 163.83 99.06 0)
+      (effects (font (size 1.27 1.27)) hide)
+    )
+    (property "Manuf" "Yageo" (id 4) (at 166.37 101.092 0)
+      (effects (font (size 1.27 1.27)) hide)
+    )
+    (property "ManufPN" "RC0603FR-071KL" (id 5) (at 166.37 101.092 0)
+      (effects (font (size 1.27 1.27)) hide)
+    )
+    (property "Supplier" "Digikey" (id 6) (at 166.37 101.092 0)
+      (effects (font (size 1.27 1.27)) hide)
+    )
+    (property "SupplierPN" "311-1.00KHRCT-ND" (id 7) (at 166.37 101.092 0)
+      (effects (font (size 1.27 1.27)) hide)
+    )
+    (pin "1")
+    (pin "2")
+  )
   (symbol (lib_id "openlst-hw:R") (at 163.83 104.14 270) (unit 1)
     (in_bom yes) (on_board yes)
@@
       (effects (font (size 1.27 1.27)) hide)
     )
-    (property "Manuf" "Samsung" (id 4) (at 107.95 90.17 0)
+    (property "Manuf" "Yageo" (id 4) (at 107.95 90.17 0)
       (effects (font (size 1.27 1.27)) hide)
     )
-    (property "ManufPN" "CL05C3R9CB5NNNC" (id 5) (at 107.95 90.17 0)
+    (property "ManufPN" "AC0402CRNPO9BN3R9" (id 5) (at 107.95 90.17 0)
       (effects (font (size 1.27 1.27)) hide)
     )
@@
       (effects (font (size 1.27 1.27)) hide)
     )
-    (property "SupplierPN" "1276-1695-1-ND" (id 7) (at 107.95 90.17 0)
+    (property "SupplierPN" "311-3054-1-ND" (id 7) (at 107.95 90.17 0)
       (effects (font (size 1.27 1.27)) hide)
     )
@@
       (effects (font (size 1.27 1.27)) hide)
     )
-    (property "Manuf" "Samsung" (id 4) (at 106.68 72.39 0)
+    (property "Manuf" "Yageo" (id 4) (at 106.68 72.39 0)
       (effects (font (size 1.27 1.27)) hide)
     )
-    (property "ManufPN" "CL05C3R9CB5NNNC" (id 5) (at 106.68 72.39 0)
+    (property "ManufPN" "AC0402CRNPO9BN3R9" (id 5) (at 106.68 72.39 0)
       (effects (font (size 1.27 1.27)) hide)
     )
@@
       (effects (font (size 1.27 1.27)) hide)
     )
-    (property "SupplierPN" "1276-1695-1-ND" (id 7) (at 106.68 72.39 0)
+    (property "SupplierPN" "311-3054-1-ND" (id 7) (at 106.68 72.39 0)
       (effects (font (size 1.27 1.27)) hide)
     )
@@
     (pin "2")
   )
+  (symbol (lib_id "openlst-hw:Ferrite_Bead") (at 250.19 41.91 0) (unit 1)
+    (in_bom yes) (on_board yes)
+    (property "Reference" "L2" (id 0) (at 246.38 41.275 90))
+    (property "Value" "Z=1k @ 100M" (id 1) (at 259.08 39.37 0))
+    (property "Footprint" "Inductor_SMD:L_0603_1608Metric" (id 2) (at 248.412 41.91 90)
+      (effects (font (size 1.27 1.27)) hide)
+    )
+    (property "Datasheet" "" (id 3) (at 250.19 41.91 0)
+      (effects (font (size 1.27 1.27)) hide)
+    )
+    (property "Manuf" "Pulse Electronics Network" (id 4) (at 250.19 41.91 90)
+      (effects (font (size 1.524 1.524)) hide)
+    )
+    (property "ManufPN" "PE-0603FB102ST" (id 5) (at 250.19 41.91 90)
+      (effects (font (size 1.524 1.524)) hide)
+    )
+    (property "Supplier" "Digikey" (id 6) (at 250.19 41.91 90)
+      (effects (font (size 1.524 1.524)) hide)
+    )
+    (property "SupplierPN" "553-2381-1-ND" (id 7) (at 250.19 41.91 90)
+      (effects (font (size 1.524 1.524)) hide)
+    )
+    (pin "1")
+    (pin "2")
+  )
   (symbol (lib_id "openlst-hw:Conn_01x03") (at 77.47 30.48 180) (unit 1)
     (in_bom yes) (on_board yes)
@@
       (effects (font (size 1.27 1.27)) hide)
     )
+    (property "SupplierPN" "SMA-J-P-H-ST-EM1" (id 7) (at 264.16 88.9 0)
+      (effects (font (size 1.27 1.27)) hide)
+    )
     (pin "1")
     (pin "2")
@@
       (effects (font (size 1.524 1.524)))
     )
-    (property "Value" "APX803S00" (id 1) (at 115.57 140.97 0)
+    (property "Value" "MIC803" (id 1) (at 132.08 130.81 0)
       (effects (font (size 1.524 1.524)))
     )
@@
       (effects (font (size 1.524 1.524)) hide)
     )
-    (property "Datasheet" "https://www.ti.com/lit/ds/symlink/tlv803.pdf" (id 3) (at 124.46 133.35 0)
+    (property "Datasheet" "https://ww1.microchip.com/downloads/en/DeviceDoc/MIC803-3-Pin-Microprocessor-Supervisor-Circuit-with-Open-Drain-Reset-Output-DS20006456A.pdf" (id 3) (at 124.46 133.35 0)
       (effects (font (size 1.524 1.524)) hide)
     )
-    (property "Manuf" "Diodes Inc" (id 4) (at 124.46 133.35 0)
+    (property "Manuf" "Microchip" (id 4) (at 124.46 133.35 0)
       (effects (font (size 1.524 1.524)) hide)
     )
-    (property "ManufPN" "APX803S00-29SR-7" (id 5) (at 124.46 133.35 0)
+    (property "ManufPN" "MIC803-29D3VM3-TR" (id 5) (at 124.46 133.35 0)
       (effects (font (size 1.524 1.524)) hide)
     )
@@
       (effects (font (size 1.524 1.524)) hide)
     )
-    (property "SupplierPN" "APX803S00-29SR-7DICT-ND" (id 7) (at 124.46 133.35 0)
+    (property "SupplierPN" "576-3804-1-ND" (id 7) (at 124.46 133.35 0)
       (effects (font (size 1.524 1.524)) hide)
     )
@@
       (effects (font (size 1.27 1.27)) hide)
     )
-    (property "Supplier" "Digikey Marketplace" (id 6) (at 201.93 38.1 0)
+    (property "Supplier" "Mouser" (id 6) (at 201.93 38.1 0)
       (effects (font (size 1.27 1.27)) hide)
     )
@@
       (reference "L1") (unit 1) (value "10u") (footprint "Inductor_SMD:L_Vishay_IFSC-1515AH_4x4x1.8mm")
     )
+    (path "/0d5ca4a9-131a-4112-97b9-bf8ae22a76ca"
+      (reference "L2") (unit 1) (value "Z=1k @ 100M") (footprint "Inductor_SMD:L_0603_1608Metric")
+    )
     (path "/00000000-0000-0000-0000-00005b333ccf"
       (reference "L3") (unit 1) (value "Z=1k @ 100M") (footprint "Inductor_SMD:L_0603_1608Metric")
@@
     )
     (path "/00000000-0000-0000-0000-00005a9a1fb1"
-      (reference "U5") (unit 1) (value "APX803S00") (footprint "Package_TO_SOT_SMD:SOT-23")
+      (reference "U5") (unit 1) (value "MIC803") (footprint "Package_TO_SOT_SMD:SOT-23")
     )
     (path "/7106b4c6-df93-4c39-8f93-ec95a19aae47"

Commit message: Started OpenLST PCB
Parts:
- U3: footprint Package_SO:SOIC-8-1EP_3.9x4.9mm_P1.27mm_EP2.62x3.51mm_ThermalVias -> openlst:SOIC-8-1EP_3.9x4.9mm_P1.27mm_EP2.613x3.502mm
Connections:
- net VAA_FILT: now reaches C11.1, C44.1, C46.1, C8.1, L2.2, U9.17 (VCC_RX), U9.26 (VCC_TX)
Changed lines of the file:
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@@
     (effects (font (size 1.524 1.524)) (justify right bottom))
   )
+  (label "VAA_FILT" (at 251.46 48.26 0)
+    (effects (font (size 1.524 1.524)) (justify left bottom))
+  )
   (symbol (lib_id "openlst-hw:+3.3V") (at 15.24 129.54 0) (unit 1)
     (in_bom yes) (on_board yes)
@@
     (property "Reference" "U3" (id 0) (at 63.5 153.67 0))
     (property "Value" "AP6502" (id 1) (at 63.5 156.21 0))
-    (property "Footprint" "Package_SO:SOIC-8-1EP_3.9x4.9mm_P1.27mm_EP2.62x3.51mm_ThermalVias" (id 2) (at 80.01 184.15 0)
+    (property "Footprint" "openlst:SOIC-8-1EP_3.9x4.9mm_P1.27mm_EP2.613x3.502mm" (id 2) (at 80.01 184.15 0)
       (effects (font (size 1.27 1.27)) hide)
     )
@@
     )
     (path "/9779f1e9-584e-4f69-b2e0-010bb1417da8"
-      (reference "U3") (unit 1) (value "AP6502") (footprint "Package_SO:SOIC-8-1EP_3.9x4.9mm_P1.27mm_EP2.62x3.51mm_ThermalVias")
+      (reference "U3") (unit 1) (value "AP6502") (footprint "openlst:SOIC-8-1EP_3.9x4.9mm_P1.27mm_EP2.613x3.502mm")
     )
     (path "/00000000-0000-0000-0000-00005b2892be"
